File: project/project.kicad_pcb (KiCad board)
At the start: 2 copper layers, 20 x 20.6 mm, 3 parts

Commit message: output_path
Parts:
- added G1: LOGO_KMS, -qr:QR, F.Cu at (174.8, 119.9)
- moved G2 5.18 mm to (174.0, 108.7)
