File: project/project.kicad_sch (KiCad schematic)
At the start: 1 part

Commit message: output_path
Parts:
- added G1: LOGO_KMS, -qr:QR, symbol -local:LOGO_KMS
Changed lines of the file:
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@@
   (symbol (lib_id "-local:LOGO_KMS") (at 157.48 180.34 0) (unit 1)
     (in_bom yes) (on_board yes) (fields_autoplaced)
-    (property "Reference" "#G1" (id 0) (at 157.48 166.4123 0)
+    (property "Reference" "G1" (id 0) (at 157.48 166.4123 0)
       (effects (font (size 1.27 1.27)) hide)
     )
@@
       (effects (font (size 1.27 1.27)) hide)
     )
-    (property "Footprint" "" (id 2) (at 157.48 180.34 0)
+    (property "Footprint" "-qr:QR" (id 2) (at 157.48 180.34 0)
       (effects (font (size 1.27 1.27)) hide)
     )
@@
   (symbol_instances
     (path "/4170c982-7626-48b7-b62a-1f9e2fa7e5fc"
-      (reference "#G1") (unit 1) (value "LOGO_KMS") (footprint "")
+      (reference "G1") (unit 1) (value "LOGO_KMS") (footprint "-qr:QR")
     )
     (path "/62316d7f-2776-43b9-a5e7-49fa1178d68c"
